File: HW/POE_5v.kicad_sch (KiCad schematic)
At the start: 60 parts, among them U1 LM5180, U11 TPS2375-1

Commit message: cleaned up and added missing files
Parts:
- C55, R50: now not fitted
Changed lines of the file:
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@@
 		(in_bom yes)
 		(on_board yes)
-		(dnp no)
+		(dnp yes)
 		(property "Reference" "R50"
 			(at 95.25 109.2199 0)
@@
 		(in_bom yes)
 		(on_board yes)
-		(dnp no)
+		(dnp yes)
 		(property "Reference" "C55"
 			(at 93.472 98.298 0)
